File: Schaltplan/SkyVision/power.kicad_sch (KiCad schematic)
At the start: 6 parts, among them CON1 SW_SPST

Commit message: wip sortieren
Parts:
- added C7: C_Polarized, symbol Device:C_Polarized
- added U3: AMS1117-3.3, Package_TO_SOT_SMD:SOT-223-3_TabPin2, symbol Regulator_Linear:AMS1117-3.3
Connections:
- net 12V: now also U3.3 (VI)
- net GND: now also C7.2, U3.1 (GND)
- new net 5V: C7.1, U3.2 (VO)
