File: Schaltplan/SkyVision/SkyVision.kicad_sch (KiCad schematic)
At the start: 18 parts, among them CON1 SW_SPST, J2 HBX, J3 DEC, J4 ST4, U1 PIC16F690-ISO, U3 AMS1117-3.3

Commit message: skyvision board weitere verkabelung vermessen.
Parts:
- added C1, C2, C3, C4, C8, C9: C, symbol Device:C
- added E1: Encoder, symbol Connector:Conn_01x07_Pin
- added M1: Motor_DC, symbol Motor:Motor_DC
- added Q1: 4947A, Package_SO:SOIC-8_3.9x4.9mm_P1.27mm, symbol Transistor_FET:IRF7309IPBF
- added Q4: 4936A, Package_SO:SOIC-8_3.9x4.9mm_P1.27mm, symbol Transistor_FET:FDS6930A
- added R1, R10 (x2), R11 (x2), R12 (x2), R13 (x2), R14, R16, R18, R2, R20, R21, R22, R23, R24, R3, R4, R5, R6, R7, R8 (x2): R, symbol Device:R
- added U4: TC4426xOA, Package_SO:SOIC-8_3.9x4.9mm_P1.27mm, symbol Driver_FET:TC4426xOA
- added X1: Crystal 20kHz, symbol Device:Crystal
- R26: value R -> 200
- renumbered C1 to C0, C2 to C7
Connections:
- net GND: now also J4.1, J4.2, C1.2, C2.2, C3.2, C8.2, C9.2, E1.2 (Pin_2), E1.5 (Pin_5), E1.6 (Pin_6), R14.1, R2.1, R7.1, U4.3 (GND)
- net at C0.1, D1.1 (K), J2.7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: no longer J2.4, J3.4, R17.1
- net at C6.1, L1.2, R26.1: now also R5.1, R6.1
- net at C7.1, U1.1 (VDD), U3.2 (VO): now also C8.1, E1.3 (Pin_3), R1.2, R10.2, R12.2, R16.2, R18.2, R22.2
- net at U1.2 (T1CKI/OSC1/CLKIN/RA5): now also C2.1, X1.1
- net at U1.3 (~{T1G}/OSC2/CLKOUT/AN3/RA4): now also C3.1, X1.2
- net at U1.4 (Vpp/~{MCLR}/RA3): now also C1.1, R1.1
- net at U1.5 (RC5/CCP1/P1A): now also Q4.4 (G2), R2.2, R4.1
- net at U1.6 (RC4/C2OUT/P1B): now also Q4.2 (G1), R3.2
- net at U1.7 (RC3/AN7/C12IN3-/P1C): now also C9.1, R20.2
- net at U1.8 (RC6/AN8/~{SS}): now also R21.2
- net at U1.9 (RC7/AN9/SDO): now also R12.2
- net at C6.2: now also R23.2, R24.1
- net at J4.3: now also R22.1
- net at J4.4: now also R11.1, R12.1
- net at J4.5: now also R8.1
- net at J4.6: now also R10.1
- net at D2.1 (K): now also R14.2
- net at R26.2: now also R21.1, R24.2
- new net: Q1.1 (S), Q1.3 (1), U4.6 (VDD)
- new net: Q1.4 (G), R6.2, U4.5 (~{OUT_B})
- new net: C4.2, M1.1 (+), Q1.5 (D), Q1.6 (D), Q4.7 (D1), Q4.8 (D1)
- new net: R4.2, U4.4 (IN_B)
- new net: Q1.2 (G), R5.2, U4.7 (~{OUT_A})
- new net: M1.2 (-), Q1.7 (D), Q1.8 (D), Q4.5 (D2), Q4.6 (D2), R8.2
- new net: E1.7 (Pin_7), R18.1
- new net: J2.4, J3.4, R17.1
- new net: C4.1, R8.1
- new net: R3.1, R7.2, U4.2 (IN_A)
- new net: Q4.1 (S1), R20.1
- new net: E1.1 (Pin_1), R16.1
- new net: E1.4 (Pin_4), R13.2
- new net: R12.1, R13.1
- new net: Q4.3 (S2), R23.1
Other:
- moved on the sheet: C6, L1, R17, R26, R9, U1

Commit message: started sorting out schematics
Parts:
- added pad: PGD, symbol Connector:Conn_01x01_Pin
- added pad: PGC, symbol Connector:Conn_01x01_Pin
Connections:
- net at C7.1, C8.1, E1.3 (Pin_3)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: now also R11.2, R8.2
- net at R13.1: now also J4.3, R22.1
- net at R13.2: now also U1.16 (RC0/AN4/C2IN+)
- net at U1.11 (SCK/SCL/RB6): now also E1.4 (Pin_4), R13.2
- net at U1.13 (SDI/SDA/AN10/RB4): now also E1.1 (Pin_1), R16.1
- net at U1.14 (RC2/AN6/C12IN2-/P1D): now also R10.2
- net at U1.15 (RC1/AN5/C12IN1-): now also R11.2
- net at U1.18 (C12IN0-/ICSPCLK/Vref/AN1/RA1): now also pad.1 (Pin_1)
- net at U1.19 (C1IN+/ICSPDAT/ULPWU/AN0/RA0): now also pad.1 (Pin_1)
- net at J4.5, R8.1: now also R11.1
- net at J4.6, R10.1: now also R10.1
Other:
- moved on the sheet: J4, R10, R11, R12, R13

Commit message: Schaltplan aufgeräumt
Changed lines of the file:
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@@
 (kicad_sch
-	(version 20231120)
+	(version 20250114)
 	(generator "eeschema")
-	(generator_version "8.0")
+	(generator_version "9.0")
 	(paper "A3")
 	(junction
@@
 	)
 	(junction
+		(at 66.04 166.37)
+		(diameter 0)
+		(color 0 0 0 0)
+	)
+	(junction
 		(at 332.74 87.63)
 		(diameter 0)
@@
 	)
 	(junction
-		(at 66.04 171.45)
-		(diameter 0)
-		(color 0 0 0 0)
-	)
-	(junction
 		(at 111.76 110.49)
 		(diameter 0)
@@
 	)
 	(junction
+		(at 66.04 168.91)
+		(diameter 0)
+		(color 0 0 0 0)
+	)
+	(junction
 		(at 91.44 52.07)
 		(diameter 0)
@@
 		(color 0 0 0 0)
 	)
+	(junction
+		(at 66.04 171.45)
+		(diameter 0)
+		(color 0 0 0 0)
+	)
 	(wire
 		(pts
@@
 	(wire
 		(pts
+			(xy 66.04 171.45) (xy 66.04 181.61)
+		)
+		(stroke
+			(width 0)
+			(type default)
+		)
+	)
+	(wire
+		(pts
 			(xy 81.28 52.07) (xy 81.28 54.61)
 		)
@@
 	(wire
 		(pts
-			(xy 63.5 166.37) (xy 72.39 166.37)
+			(xy 63.5 166.37) (xy 66.04 166.37)
 		)
 		(stroke
@@
 	(wire
 		(pts
-			(xy 66.04 168.91) (xy 66.04 171.45)
-		)
-		(stroke
-			(width 0)
-			(type default)
-		)
-	)
-	(wire
-		(pts
 			(xy 48.26 133.35) (xy 60.96 133.35)
 		)
@@
 	(wire
 		(pts
-			(xy 66.04 171.45) (xy 66.04 181.61)
+			(xy 105.41 38.1) (xy 116.84 38.1)
 		)
 		(stroke
@@
 	(wire
 		(pts
-			(xy 105.41 38.1) (xy 116.84 38.1)
+			(xy 346.71 40.64) (xy 346.71 22.86)
 		)
 		(stroke
@@
 	(wire
 		(pts
-			(xy 346.71 40.64) (xy 346.71 22.86)
+			(xy 31.75 171.45) (xy 54.61 171.45)
 		)
 		(stroke
@@
 	(wire
 		(pts
-			(xy 31.75 171.45) (xy 54.61 171.45)
+			(xy 63.5 181.61) (xy 63.5 267.97)
 		)
 		(stroke
@@
 	(wire
 		(pts
-			(xy 63.5 181.61) (xy 63.5 267.97)
+			(xy 222.25 200.66) (xy 227.33 200.66)
 		)
 		(stroke
@@
 	(wire
 		(pts
-			(xy 222.25 200.66) (xy 227.33 200.66)
+			(xy 124.46 205.74) (xy 109.22 205.74)
 		)
 		(stroke
@@
 	(wire
 		(pts
-			(xy 124.46 205.74) (xy 109.22 205.74)
+			(xy 66.04 166.37) (xy 72.39 166.37)
 		)
 		(stroke
@@
 	(wire
 		(pts
+			(xy 66.04 166.37) (xy 66.04 168.91)
+		)
+		(stroke
+			(width 0)
+			(type default)
+		)
+	)
+	(wire
+		(pts
 			(xy 46.99 87.63) (xy 68.58 87.63)
 		)
@@
 	(wire
 		(pts
+			(xy 66.04 168.91) (xy 66.04 171.45)
+		)
+		(stroke
+			(width 0)
+			(type default)
+		)
+	)
+	(wire
+		(pts
 			(xy 48.26 123.19) (xy 48.26 118.11)
 		)
@@
 		)
 	)
+	(embedded_fonts no)
 )
