File: Schaltplan/SkyVision/motor.kicad_sch (KiCad schematic)
At the start: 0 parts

Commit message: Schaltplan aufgeräumt
Parts:
- added C4: C, symbol Device:C
- added C6: C_Polarized, symbol Device:C_Polarized
- added L1: L, symbol Device:L
- added M1: Motor_DC, symbol Motor:Motor_DC
- added Q1: 4947A, Package_SO:SOIC-8_3.9x4.9mm_P1.27mm, symbol Transistor_FET:IRF7309IPBF
- added Q4: 4936A, Package_SO:SOIC-8_3.9x4.9mm_P1.27mm, symbol Transistor_FET:FDS6930A
- added R2, R23, R24, R3, R4, R5, R6, R7, R8: R, symbol Device:R
- added R26: 200, symbol Device:R
- added U4: TC4426xOA, Package_SO:SOIC-8_3.9x4.9mm_P1.27mm, symbol Driver_FET:TC4426xOA
Connections:
- new net: Q1.1 (S), Q1.3 (1), U4.6 (VDD)
- new net: Q1.4 (G), R6.2, U4.5 (~{OUT_B})
- new net: C4.1, M1.1 (+), Q1.5 (D), Q1.6 (D), Q4.7 (D1), Q4.8 (D1)
- new net: C6.1, L1.2, R26.2, R5.1, R6.1
- new net: R2.1, R4.2, U4.4 (IN_B)
- new net: Q1.2 (G), R5.2, U4.7 (~{OUT_A})
- new net: M1.2 (-), Q1.7 (D), Q1.8 (D), Q4.5 (D2), Q4.6 (D2), R8.1
- new net: C4.2, R8.2
- new net: C6.2, R23.2, R24.1
- new net: R3.1, R7.2, U4.2 (IN_A)
- new net: Q4.3 (S2), R23.1
- new net 12V: L1.1
- new net GND: R2.2, R7.1, U4.3 (GND)
- new net RC3: Q4.1 (S1)
- new net RC4: Q4.2 (G1), R3.2
- new net RC5: Q4.4 (G2), R4.1
- new net RC6: R24.2, R26.1
