File: Schaltplan/Pico_Joystick_Control/pico_control/pico_control.kicad_sch (KiCad schematic)
At the start: 7 parts, among them J1 RJ45, J3 RJ12, U1 TXB0104D, U2 TBA1-1211

Commit message: rpi zero addad to scheme
Parts:
- added U4: RASPBERRY_PI_ZERO_2_W, RASPBERRY_PI_ZERO_2_W:MODULE_RASPBERRY_PI_ZERO_2_W, symbol RASPBERRY_PI_ZERO_2_W:RASPBERRY_PI_ZERO_2_W
